Commit message: resized wheels and chassis

File: urdf/robot.xacro (robot description, xacro)
@@ -7,19 +7,19 @@
     <link name="link_chassis">
         <inertial>
-            <mass value="5" />
-            <origin xyz="0 0 0.3" rpy="0 0 0" />
+            <mass value="1" />
+            <origin xyz="0 0 0.2" rpy="0 0 0" />
             <inertia ixx="1.5417" ixy="0" ixz="0" iyy="3.467" iyz="0" izz="4.742" />
         </inertial>
         <collision>
             <geometry>
-                <box size="2 1.3 0.4" />
+                <box size="1 0.75 0.2" />
             </geometry>
         </collision>
         <visual>
             <geometry>
-                <box size="2 1.3 0.4" />
+                <box size="1 0.75 0.2" />
             </geometry>
-            <material name="Blue">
-                <color rgba="0 0 1 1" />
+            <material name="Red">
+                <color rgba="1 0 0 1" />
             </material>
         </visual>
@@ -27,5 +27,5 @@
     <!-- Joint - chassis / left wheel -->
     <joint name="joint_chassis_left_wheel" type="continuous">
-        <origin rpy="0 0 0" xyz="-0.5 0.65 0" />
+        <origin rpy="0 0 0" xyz="-0.3 0.375 0" />
         <child link="link_left_wheel" />
         <parent link="link_chassis" />
@@ -37,18 +37,18 @@
     <link name="link_left_wheel">
         <inertial>
-            <mass value="1" />
+            <mass value="0.5" />
             <origin xyz="0 0 0" rpy="0 0 0" />
             <inertia ixx="0.002526666666667" ixy="0" ixz="0" iyy="0.002526666666667" iyz="0" izz="0.005"/>
         </inertial>
         <collision>
-            <origin rpy="${pi / 2} 0 0" xyz="0 0.18 0" />
+            <origin rpy="${pi / 2} 0 0" xyz="0 0.1 0" />
             <geometry>
-                <cylinder length="0.12" radius="0.4"/>
+                <cylinder length="0.1" radius="0.25"/>
             </geometry>
         </collision>
         <visual>
-            <origin rpy="${pi / 2} 0 0" xyz="0 0.18 0" />
+            <origin rpy="${pi / 2} 0 0" xyz="0 0.1 0" />
             <geometry>
-                <mesh filename="package://robot_description/meshes/wheel.stl" />
+                <mesh filename="package://robot_description/meshes/wheel.stl" scale="0.5 0.5 0.5" />
             </geometry>
             <material name="Black">
@@ -57,31 +57,31 @@
         </visual>
         <collision>
-            <origin rpy="${pi / 2} 0 0" xyz="0 0.06 0" />
+            <origin rpy="${pi / 2} 0 0" xyz="0 0.0525 0" />
             <geometry>
-                <cylinder length="0.18" radius="0.08"/>
+                <cylinder length="0.105" radius="0.05"/>
             </geometry>
         </collision>
         <visual>
-            <origin rpy="${pi / 2} 0 0" xyz="0 0.06 0" />
+            <origin rpy="${pi / 2} 0 0" xyz="0 0.0525 0" />
             <geometry>
-                <cylinder length="0.18" radius="0.08"/>
+                <cylinder length="0.105" radius="0.05"/>
             </geometry>
-            <material name="White">
-                <color rgba="1 1 1 1" />
+            <material name="Black">
+                <color rgba="0 0 0 1" />
             </material>
         </visual>
         <collision>
-            <origin rpy="${pi / 2} 0 0" xyz="0 0.18 0" />
+            <origin rpy="${pi} 0 0" xyz="0 0.1 0" />
             <geometry>
-                <box size="0.03 0.01 0.6" />
+                <box size="0.03 0.01 0.3" />
             </geometry>
         </collision>
         <visual>
-            <origin rpy="${pi / 2} 0 0" xyz="0 0.18 0" />
+            <origin rpy="${pi} 0 0" xyz="0 0.1 0" />
             <geometry>
-                <box size="0.03 0.01 0.6" />
+                <box size="0.03 0.01 0.3" />
             </geometry>
-            <material name="White">
-                <color rgba="1 1 1 1" />
+            <material name="Black">
+                <color rgba="0 0 0 1" />
             </material>
         </visual>
@@ -89,5 +89,5 @@
     <!-- Joint - chassis / right wheel -->
     <joint name="joint_chassis_right_wheel" type="continuous">
-        <origin rpy="0 0 0" xyz="-0.5 -0.65 0" />
+        <origin rpy="0 0 0" xyz="-0.3 -0.375 0" />
         <child link="link_right_wheel" />
         <parent link="link_chassis" />
@@ -99,18 +99,18 @@
     <link name="link_right_wheel">
         <inertial>
-            <mass value="1" />
+            <mass value="0.5" />
             <origin xyz="0 0 0" rpy="0 0 0" />
             <inertia ixx="0.002526666666667" ixy="0" ixz="0" iyy="0.002526666666667" iyz="0" izz="0.005"/>
         </inertial>
         <collision>
-            <origin rpy="${pi / 2} 0 0" xyz="0 -0.18 0" />
+            <origin rpy="${pi / 2} 0 0" xyz="0 -0.1 0" />
             <geometry>
-                <cylinder length="0.12" radius="0.4"/>
+                <cylinder length="0.1" radius="0.25"/>
             </geometry>
         </collision>
         <visual>
-            <origin rpy="${pi / 2} 0 0" xyz="0 -0.18 0" />
+            <origin rpy="${pi / 2} 0 0" xyz="0 -0.1 0" />
             <geometry>
-                <mesh filename="package://robot_description/meshes/wheel.stl" />
+                <mesh filename="package://robot_description/meshes/wheel.stl" scale="0.5 0.5 0.5" />
             </geometry>
             <material name="Black">
@@ -119,31 +119,31 @@
         </visual>
         <collision>
-            <origin rpy="${pi / 2} 0 0" xyz="0 -0.06 0" />
+            <origin rpy="${pi / 2} 0 0" xyz="0 -0.0525 0" />
             <geometry>
-                <cylinder length="0.18" radius="0.08"/>
+                <cylinder length="0.105" radius="0.05"/>
             </geometry>
         </collision>
         <visual>
-            <origin rpy="${pi / 2} 0 0" xyz="0 -0.06 0" />
+            <origin rpy="${pi / 2} 0 0" xyz="0 -0.0525 0" />
             <geometry>
-                <cylinder length="0.18" radius="0.08"/>
+                <cylinder length="0.105" radius="0.05"/>
             </geometry>
-            <material name="White">
-                <color rgba="1 1 1 1" />
+            <material name="Black">
+                <color rgba="0 0 0 1" />
             </material>
         </visual>
         <collision>
-            <origin rpy="${pi / 2} 0 0" xyz="0 -0.18 0" />
+            <origin rpy="${pi} 0 0" xyz="0 -0.1 0" />
             <geometry>
-                <box size="0.03 0.01 0.6" />
+                <box size="0.03 0.01 0.3" />
             </geometry>
         </collision>
         <visual>
-            <origin rpy="${pi / 2} 0 0" xyz="0 -0.18 0" />
+            <origin rpy="${pi} 0 0" xyz="0 -0.1 0" />
             <geometry>
-                <box size="0.03 0.01 0.6" />
+                <box size="0.03 0.01 0.3" />
             </geometry>
-            <material name="White">
-                <color rgba="1 1 1 1" />
+            <material name="Black">
+                <color rgba="0 0 0 1" />
             </material>
         </visual>

Commit message: modified joint and link names to capture 4 wheel robot and created two front wheels

File: urdf/robot.xacro (robot description, xacro)
@@ -25,8 +25,8 @@
         </visual>
     </link>
-    <!-- Joint - chassis / left wheel -->
-    <joint name="joint_chassis_left_wheel" type="continuous">
+    <!-- Joint - chassis / rear left wheel -->
+    <joint name="joint_chassis_rear_left_wheel" type="continuous">
         <origin rpy="0 0 0" xyz="-0.3 0.375 0" />
-        <child link="link_left_wheel" />
+        <child link="link_rear_left_wheel" />
         <parent link="link_chassis" />
         <axis rpy="0 0 0" xyz="0 1 0" />
@@ -34,6 +34,6 @@
         <joint_properties damping="1.0" friction="1.0" />
     </joint>
-    <!-- Link - left wheel -->
-    <link name="link_left_wheel">
+    <!-- Link - rear left wheel -->
+    <link name="link_rear_left_wheel">
         <inertial>
             <mass value="0.5" />
@@ -87,8 +87,8 @@
         </visual>
     </link>
-    <!-- Joint - chassis / right wheel -->
-    <joint name="joint_chassis_right_wheel" type="continuous">
-        <origin rpy="0 0 0" xyz="-0.3 -0.375 0" />
-        <child link="link_right_wheel" />
+    <!-- Joint - chassis / front left wheel -->
+    <joint name="joint_chassis_front_left_wheel" type="continuous">
+        <origin rpy="0 0 0" xyz="0.3 0.375 0" />
+        <child link="link_front_left_wheel" />
         <parent link="link_chassis" />
         <axis rpy="0 0 0" xyz="0 1 0" />
@@ -96,6 +96,130 @@
         <joint_properties damping="1.0" friction="1.0" />
     </joint>
-    <!-- Link - right wheel -->
-    <link name="link_right_wheel">
+    <!-- Link - front left wheel -->
+    <link name="link_front_left_wheel">
+        <inertial>
+            <mass value="0.5" />
+            <origin xyz="0 0 0" rpy="0 0 0" />
+            <inertia ixx="0.002526666666667" ixy="0" ixz="0" iyy="0.002526666666667" iyz="0" izz="0.005"/>
+        </inertial>
+        <collision>
+            <origin rpy="${pi / 2} 0 0" xyz="0 0.1 0" />
+            <geometry>
+                <cylinder length="0.1" radius="0.25"/>
+            </geometry>
+        </collision>
+        <visual>
+            <origin rpy="${pi / 2} 0 0" xyz="0 0.1 0" />
+            <geometry>
+                <mesh filename="package://robot_description/meshes/wheel.stl" scale="0.5 0.5 0.5" />
+            </geometry>
+            <material name="Black">
+                <color rgba="0 0 0 1" />
+            </material>
+        </visual>
+        <collision>
+            <origin rpy="${pi / 2} 0 0" xyz="0 0.0525 0" />
+            <geometry>
+                <cylinder length="0.105" radius="0.05"/>
+            </geometry>
+        </collision>
+        <visual>
+            <origin rpy="${pi / 2} 0 0" xyz="0 0.0525 0" />
+            <geometry>
+                <cylinder length="0.105" radius="0.05"/>
+            </geometry>
+            <material name="Black">
+                <color rgba="0 0 0 1" />
+            </material>
+        </visual>
+        <collision>
+            <origin rpy="${pi} 0 0" xyz="0 0.1 0" />
+            <geometry>
+                <box size="0.03 0.01 0.3" />
+            </geometry>
+        </collision>
+        <visual>
+            <origin rpy="${pi} 0 0" xyz="0 0.1 0" />
+            <geometry>
+                <box size="0.03 0.01 0.3" />
+            </geometry>
+            <material name="Black">
+                <color rgba="0 0 0 1" />
+            </material>
+        </visual>
+    </link>
+    <!-- Joint - chassis / rear right wheel -->
+    <joint name="joint_chassis_rear_right_wheel" type="continuous">
+        <origin rpy="0 0 0" xyz="-0.3 -0.375 0" />
+        <child link="link_rear_right_wheel" />
+        <parent link="link_chassis" />
+        <axis rpy="0 0 0" xyz="0 1 0" />
+        <limit effort="10000" velocity="1000" />
+        <joint_properties damping="1.0" friction="1.0" />
+    </joint>
+    <!-- Link - rear right wheel -->
+    <link name="link_rear_right_wheel">
+        <inertial>
+            <mass value="0.5" />
+            <origin xyz="0 0 0" rpy="0 0 0" />
+            <inertia ixx="0.002526666666667" ixy="0" ixz="0" iyy="0.002526666666667" iyz="0" izz="0.005"/>
+        </inertial>
+        <collision>
+            <origin rpy="${pi / 2} 0 0" xyz="0 -0.1 0" />
+            <geometry>
+                <cylinder length="0.1" radius="0.25"/>
+            </geometry>
+        </collision>
+        <visual>
+            <origin rpy="${pi / 2} 0 0" xyz="0 -0.1 0" />
+            <geometry>
+                <mesh filename="package://robot_description/meshes/wheel.stl" scale="0.5 0.5 0.5" />
+            </geometry>
+            <material name="Black">
+                <color rgba="0 0 0 1" />
+            </material>
+        </visual>
+        <collision>
+            <origin rpy="${pi / 2} 0 0" xyz="0 -0.0525 0" />
+            <geometry>
+                <cylinder length="0.105" radius="0.05"/>
+            </geometry>
+        </collision>
+        <visual>
+            <origin rpy="${pi / 2} 0 0" xyz="0 -0.0525 0" />
+            <geometry>
+                <cylinder length="0.105" radius="0.05"/>
+            </geometry>
+            <material name="Black">
+                <color rgba="0 0 0 1" />
+            </material>
+        </visual>
+        <collision>
+            <origin rpy="${pi} 0 0" xyz="0 -0.1 0" />
+            <geometry>
+                <box size="0.03 0.01 0.3" />
+            </geometry>
+        </collision>
+        <visual>
+            <origin rpy="${pi} 0 0" xyz="0 -0.1 0" />
+            <geometry>
+                <box size="0.03 0.01 0.3" />
+            </geometry>
+            <material name="Black">
+                <color rgba="0 0 0 1" />
+            </material>
+        </visual>
+    </link>
+    <!-- Joint - chassis / front right wheel -->
+    <joint name="joint_chassis_front_right_wheel" type="continuous">
+        <origin rpy="0 0 0" xyz="0.3 -0.375 0" />
+        <child link="link_front_right_wheel" />
+        <parent link="link_chassis" />
+        <axis rpy="0 0 0" xyz="0 1 0" />
+        <limit effort="10000" velocity="1000" />
+        <joint_properties damping="1.0" friction="1.0" />
+    </joint>
+    <!-- Link - front right wheel -->
+    <link name="link_front_right_wheel">
         <inertial>
             <mass value="0.5" />

Commit message: resized laser sensor to reflect hokuyo UST-10LX model, and placed it on robot

File: urdf/robot.xacro (robot description, xacro)
@@ -8,5 +8,5 @@
         <inertial>
             <mass value="1" />
-            <origin xyz="0 0 0.2" rpy="0 0 0" />
+            <origin xyz="0 0 0" rpy="0 0 0" />
             <inertia ixx="1.5417" ixy="0" ixz="0" iyy="3.467" iyz="0" izz="4.742" />
         </inertial>
@@ -273,7 +273,7 @@
         </visual>
     </link>
-        <!-- Joint : Laser scan -->
+    <!-- Joint : Laser scan -->
     <joint name="joint_laser_scan_chassis" type="fixed">
-        <origin rpy="0 0 0" xyz="0.8 0 0.3" />
+        <origin rpy="0 0 0" xyz="0.4 0 0.135" />
         <child link="link_laser_scan" />
         <parent link="link_chassis" />
@@ -284,5 +284,5 @@
         <inertial>
             <origin xyz="0 0 0" rpy="0 0 0" />
-            <mass value="0.5" />
+            <mass value="0.25" />
             <inertia ixx="0.000252666666667" ixy="0" ixz="0" iyy="0.000252666666667" iyz="0" izz="0.0005"/>
         </inertial>
@@ -290,8 +290,8 @@
             <origin xyz="0 0 0" rpy="0 0 0" />
             <geometry>
-                <cylinder radius="0.15" length="0.20"/>
-            </geometry>
-            <material name="Red">
-                <color rgba="0.7 0.1 0.1 1" />
+                <cylinder radius="0.05" length="0.07"/>
+            </geometry>
+            <material name="Black">
+                <color rgba="0 0 0 1" />
             </material>
         </visual>
@@ -299,5 +299,5 @@
             <origin xyz="0 0 0" rpy="0 0 0"/>
             <geometry>
-                <cylinder radius="0.15" length="0.20"/>
+                <cylinder radius="0.05" length="0.07"/>
             </geometry>
         </collision>

Commit message: resized robot slightly to remove interference with laser scanner, and added a spawn.launch file to spawn the robot in GAZEBO worlds

File: urdf/robot.xacro (robot description, xacro)
@@ -27,5 +27,5 @@
     <!-- Joint - chassis / rear left wheel -->
     <joint name="joint_chassis_rear_left_wheel" type="continuous">
-        <origin rpy="0 0 0" xyz="-0.3 0.375 0" />
+        <origin rpy="0 0 0" xyz="-0.225 0.375 0" />
         <child link="link_rear_left_wheel" />
         <parent link="link_chassis" />
@@ -89,5 +89,5 @@
     <!-- Joint - chassis / front left wheel -->
     <joint name="joint_chassis_front_left_wheel" type="continuous">
-        <origin rpy="0 0 0" xyz="0.3 0.375 0" />
+        <origin rpy="0 0 0" xyz="0.225 0.375 0" />
         <child link="link_front_left_wheel" />
         <parent link="link_chassis" />
@@ -151,5 +151,5 @@
     <!-- Joint - chassis / rear right wheel -->
     <joint name="joint_chassis_rear_right_wheel" type="continuous">
-        <origin rpy="0 0 0" xyz="-0.3 -0.375 0" />
+        <origin rpy="0 0 0" xyz="-0.225 -0.375 0" />
         <child link="link_rear_right_wheel" />
         <parent link="link_chassis" />
@@ -213,5 +213,5 @@
     <!-- Joint - chassis / front right wheel -->
     <joint name="joint_chassis_front_right_wheel" type="continuous">
-        <origin rpy="0 0 0" xyz="0.3 -0.375 0" />
+        <origin rpy="0 0 0" xyz="0.225 -0.375 0" />
         <child link="link_front_right_wheel" />
         <parent link="link_chassis" />

Commit message: inherited autonomy script to improve, and modified height of laser sensor in URDF to pick up the proj_model objects in gazebo

File: urdf/robot.xacro (robot description, xacro)
@@ -16,7 +16,22 @@
             </geometry>
         </collision>
+        <collision>
+            <origin rpy="0 0 0" xyz="0.3 0 0.3" />
+            <geometry>
+                <box size="0.2 0.2 0.4" />
+            </geometry>
+        </collision>
         <visual>
             <geometry>
                 <box size="1 0.75 0.2" />
+            </geometry>
+            <material name="Red">
+                <color rgba="1 0 0 1" />
+            </material>
+        </visual>
+        <visual>
+            <origin rpy="0 0 0" xyz="0.4 0 0.3" />
+            <geometry>
+                <box size="0.2 0.2 0.4" />
             </geometry>
             <material name="Red">
@@ -275,5 +290,5 @@
     <!-- Joint : Laser scan -->
     <joint name="joint_laser_scan_chassis" type="fixed">
-        <origin rpy="0 0 0" xyz="0.4 0 0.135" />
+        <origin rpy="0 0 0" xyz="0.4 0 0.535" />
         <child link="link_laser_scan" />
         <parent link="link_chassis" />
